Commit message: Got RVIZ to show links, but in the wrong place

File: catkin_ws/src/arm_description/urdf/RobotURDF.SLDASM.urdf (robot description, URDF)
Before this commit: robot urdf, 5 links, 4 joints
Links:
- link base_link: geometry collision mesh filename=package://arm_description/meshes/base_link.STL; visual mesh filename=package://arm_description/meshes/base_link.STL
- link link_1: geometry collision mesh filename=package://arm_description/meshes/link_1.STL; visual mesh filename=package://arm_description/meshes/link_1.STL
- link link_2: geometry collision mesh filename=package://arm_description/meshes/link_2.STL; visual mesh filename=package://arm_description/meshes/link_2.STL
- link link_3: geometry collision mesh filename=package://arm_description/meshes/link_3.STL; visual mesh filename=package://arm_description/meshes/link_3.STL
